File: MicroMouse.kicad_pcb (KiCad board)
At the start: 2 copper layers, 100 x 80 mm, 81 parts, among them CN1 mouseBattery, Q1 IRLML6402, Q2 IRLML6344, SW1 SPST, SW2 SPST, SW3 SPST, U1 STM32F405RGTx, U2 TB6612, U3 CN_MOTOR, U4 CN_MOTOR, U5 3p, U6 ICM-20602, U7 4p

Commit message: pushできるかな
Parts:
- moved D4 9.16 mm to (27.9, 4.06)
- moved R8 8.68 mm to (25.9, 96.5)
- moved R5 8.65 mm to (27.9, 6.60)
- moved R7 8.64 mm to (20.8, 85.3)
- moved R6 4.68 mm to (27.4, 73.7)
- moved R2 4.19 mm to (4.06, 39.1), turned to 90 degrees
- moved C11 4.02 mm to (39.0, 42.0), turned to 180 degrees
- moved R4 3.56 mm to (7.62, 55.9), turned to 315 degrees
- moved D2 2.97 mm to (6.10, 21.3), turned to 45 degrees
- moved C12 2.17 mm to (31.0, 30.0)
- moved R11 2.14 mm to (36.0, 26.0), turned to 270 degrees
- moved R3 1.93 mm to (7.11, 22.4), turned to 45 degrees
- moved D1 1.14 mm to (2.03, 39.1), turned to 90 degrees
- moved D3 1.02 mm to (6.10, 57.4), turned to 315 degrees
- moved D5 1.02 mm to (27.4, 75.7), turned to 0 degrees
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Connections:
- U1 pad 10: LED_LF -> SEN_RS
- U1 pad 11: LED_LS -> DBG_LED_3
- U1 pad 14: Net-(U1-Pad14) -> DBG_LED_5
- U1 pad 15: Net-(U1-Pad15) -> SEN_LF
- U1 pad 16: M_PWM_R -> LED_LF
- U1 pad 17: M_PWM_L -> LED_LS
- U1 pad 2: DBG_LED_4 -> Net-(U1-Pad2)
- U1 pad 20: SEN_BAT -> SEN_LS
- U1 pad 22: R_ENC_A -> L_ENC_A
- U1 pad 23: R_ENC_B -> L_ENC_B
- U1 pad 24: M_IN1_R -> M_IN2_L
- U1 pad 26: M_IN2_L -> M_STBY
- U1 pad 27: M_IN2_R -> M_IN1_R
- U1 pad 28: M_STBY -> M_IN2_R
- U1 pad 29: SEN_RS -> M_PWM_L
- U1 pad 3: DBG_LED_5 -> Net-(U1-Pad3)
- U1 pad 30: SEN_RF -> CS
- U1 pad 33: CS -> Mode_SW
- U1 pad 37: L_ENC_A -> R_ENC_A
- U1 pad 38: L_ENC_B -> R_ENC_B
- U1 pad 44: Net-(U1-Pad44) -> M_PWM_R
- U1 pad 45: Net-(U1-Pad45) -> LED_RS
- U1 pad 50: Net-(U1-Pad50) -> LED_RF
- U1 pad 51: DBG_LED_1 -> SCL
- U1 pad 52: DBG_LED_2 -> SDO
- U1 pad 53: DBG_LED_3 -> SDA
- U1 pad 54: Net-(U1-Pad54) -> DBG_LED_4
- U1 pad 55: SCL -> Net-(U1-Pad55)
- U1 pad 56: SDO -> Net-(U1-Pad56)
- U1 pad 57: SDA -> Net-(U1-Pad57)
- U1 pad 58: SEN_LF -> Net-(U1-Pad58)
- U1 pad 59: SEN_LS -> DBG_LED_2
- U1 pad 62: Mode_SW -> DBG_LED_1
- U1 pad 8: LED_RS -> SEN_RF
- U1 pad 9: LED_RF -> SEN_BAT
Routing:
- net GND: track 280.7 -> 401.7 mm, vias 0 -> 8
- net +3V3: track 202.2 -> 173.0 mm, vias 9 -> 8
- net Net-(Q2-Pad1): track 0.00 -> 7.56 mm
- net Net-(C11-Pad2): track 0.00 -> 5.09 mm
- net Net-(Q2-Pad3): track 0.00 -> 4.21 mm
- net VCC: track 66.3 -> 70.4 mm
- net Net-(D11-Pad1): track 26.3 -> 29.3 mm
- net Net-(C12-Pad2): track 0.00 -> 2.60 mm
- net SEN_BAT: track 0.00 -> 2.00 mm
- net Net-(D11-Pad2): track 27.4 -> 29.2 mm
- net Net-(Q1-Pad1): track 9.76 -> 10.7 mm
- net Net-(D9-Pad1): track 28.6 -> 29.3 mm
- net Net-(U2-Pad11): track 0.00 -> 0.65 mm
- net Net-(U2-Pad1): track 0.00 -> 0.65 mm
- net Net-(U2-Pad7): track 0.00 -> 0.65 mm
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
Commit message: 信号線を引きたいマン
Routing:
- net GND: track 401.7 -> 448.6 mm, vias 8 -> 15
Changed lines of the file:
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@@
   (general
     (links 194)
-    (no_connects 75)
-    (area -0.050001 -0.050001 100.050001 80.050001)
+    (no_connects 69)
+    (area -0.993 -10.725 101.475 99.395)
     (thickness 1.6)
     (drawings 13)
-    (tracks 425)
+    (tracks 456)
     (zones 0)
     (modules 81)
@@
   )
   (setup
-    (last_trace_width 0.5)
+    (last_trace_width 0.7)
     (user_trace_width 0.4)
     (user_trace_width 0.5)
@@
   (segment (start 71 34.1) (end 74 34.1) (width 0.7) (layer F.Cu) (net 1))
   (segment (start 42.588 21.844) (end 42.588 21.928) (width 0.7) (layer F.Cu) (net 1))
+  (segment (start 19.812 48.26) (end 22.352 50.8) (width 0.7) (layer B.Cu) (net 2))
+  (segment (start 27.224 51.1) (end 28 51.1) (width 0.7) (layer F.Cu) (net 2) (status 800000))
+  (segment (start 26.924 50.8) (end 27.224 51.1) (width 0.7) (layer F.Cu) (net 2))
+  (via (at 26.924 50.8) (size 0.6) (drill 0.4) (layers F.Cu B.Cu) (net 2))
+  (segment (start 22.352 50.8) (end 26.924 50.8) (width 0.7) (layer B.Cu) (net 2))
+  (segment (start 15.748 40.64) (end 15.748 44.196) (width 0.7) (layer B.Cu) (net 2))
+  (segment (start 19.812 48.26) (end 20.222183 48.670183) (width 0.7) (layer F.Cu) (net 2) (status 800000))
+  (via (at 19.812 48.26) (size 0.6) (drill 0.4) (layers F.Cu B.Cu) (net 2))
+  (segment (start 15.748 44.196) (end 19.812 48.26) (width 0.7) (layer B.Cu) (net 2))
+  (segment (start 20.222183 48.670183) (end 20.222183 48.777817) (width 0.7) (layer F.Cu) (net 2) (status C00000))
+  (segment (start 15.748 38.1) (end 15.748 40.64) (width 0.7) (layer B.Cu) (net 2))
+  (segment (start 15.748 40.64) (end 15.9 40.792) (width 0.7) (layer F.Cu) (net 2) (status C00000))
+  (via (at 15.748 40.64) (size 0.6) (drill 0.4) (layers F.Cu B.Cu) (net 2) (status 800000))
+  (segment (start 15.9 40.792) (end 15.9 41) (width 0.7) (layer F.Cu) (net 2) (status C00000))
+  (segment (start 17.78 31.496) (end 15.748 33.528) (width 0.7) (layer B.Cu) (net 2))
+  (segment (start 15.9 38.252) (end 15.9 39) (width 0.7) (layer F.Cu) (net 2) (status 800000))
+  (segment (start 15.748 38.1) (end 15.9 38.252) (width 0.7) (layer F.Cu) (net 2))
+  (via (at 15.748 38.1) (size 0.6) (drill 0.4) (layers F.Cu B.Cu) (net 2))
+  (segment (start 15.748 33.528) (end 15.748 38.1) (width 0.7) (layer B.Cu) (net 2))
+  (segment (start 28.956 28.956) (end 20.32 28.956) (width 0.7) (layer B.Cu) (net 2))
+  (segment (start 17.78 31.496) (end 17.222183 32.053817) (width 0.7) (layer F.Cu) (net 2))
+  (via (at 17.78 31.496) (size 0.6) (drill 0.4) (layers F.Cu B.Cu) (net 2))
+  (segment (start 20.32 28.956) (end 17.78 31.496) (width 0.7) (layer B.Cu) (net 2))
+  (segment (start 17.222183 32.053817) (end 17.222183 32.222183) (width 0.7) (layer F.Cu) (net 2))
+  (segment (start 31 28.9) (end 30.536 28.9) (width 0.7) (layer F.Cu) (net 2))
+  (segment (start 28.9 28.9) (end 28 28.9) (width 0.7) (layer F.Cu) (net 2))
+  (segment (start 28.956 28.956) (end 28.9 28.9) (width 0.7) (layer F.Cu) (net 2))
+  (via (at 28.956 28.956) (size 0.6) (drill 0.4) (layers F.Cu B.Cu) (net 2))
+  (segment (start 30.48 28.956) (end 28.956 28.956) (width 0.7) (layer B.Cu) (net 2))
+  (via (at 30.48 28.956) (size 0.6) (drill 0.4) (layers F.Cu B.Cu) (net 2))
+  (segment (start 30.536 28.9) (end 30.48 28.956) (width 0.7) (layer F.Cu) (net 2))
   (segment (start 45.3 25) (end 45.3 25.488) (width 0.7) (layer F.Cu) (net 2))
   (segment (start 45.3 25.488) (end 50.292 30.48) (width 0.7) (layer F.Cu) (net 2))
